File: Hardware/leitorcartao.brd (EAGLE design)
At the start: 34.5 x 67 mm, 131 parts, among them IC2 TL084D, Q1 BSH103, Q2 BC847ASMD, Q3 BC857ALT1SMD, Q4 BC847ALT1SMD, Q5 BC847ALT1SMD, Q6 BC847ALT1SMD, Q7 BC847ALT1SMD, Q8 BC847ALT1SMD, U1 ATXMEGA8E5-AU, U2 AP1117IE33G-13, U3 TLV1117-50CDCYR, U4 MFRC52202HN1, X1 ANTENA 125kHz, X2 MIFARE ANTENA

Commit message: Nova versão da placa do leitor de parede. Em progesso.
Parts:
- removed L2: AIUR-02H-271K, RFiD:AIUR-02H-271K
- removed LED1: LTST-C235KGKRKT, RFiD:LTST-C235KGKRKT
- removed PROG/DBG: (no value), pinhead:1X04
- added C43: 4.7uF, RFiD:C0402
- added C44: 4.7nF, RFiD:C0402
- added C45: 22pF, RFiD:C0402
- added C46: 100n, RFiD:C0402
- added C47: 100p, RFiD:C0402
- added C48: 68p, RFiD:C0402
- added C49, C52, C53: 0.1uF, RFiD:C0402
- added C50: 68pF, RFiD:C0402
- added C51: 100pF, RFiD:C0402
- added IC1: TL084, RFiD:TSSOP14
- added JP1: (no value), pinhead:1X05
- added LED2: SMP4-SBC, RFiD:SMP4-SBC
- added R46, R47: 10, RFiD:R0603
- added R48: 68k, RFiD:R0402
- added R49: 330k, RFiD:R0402
- added R50: 10k, RFiD:R0402
- added R51, R54: 5.6k, RFiD:R0402
- added R52, R55: 5.1k, RFiD:R0402
- added R53, R56: 270k, RFiD:R0402
- C12, C13, C14, C15, C16: device RFiD:C0402 -> RFiD:C0603
- C18: value 100nF -> 220nF
- C19: value 470pF -> 220p
- C2, C3: value 100nF -> 0.1uF
- C20, C23: value 100pF -> 47p
- C21: value 1nF -> 47p
- C22: value 220nF -> 47p
- C24: value 220nF -> 47nF
- C25: value 220pF -> 4.7nF
- C26, C28: value 220pF -> 0.1uF
- C27: value 470pF -> 22pF
- C29: value 220pF -> 47nF
- C42: value 10uF -> 0.1uF
- IC2: value TL084D -> TL084; device RFiD:SO14 -> RFiD:TSSOP14
- R10: value 1k -> 27k
- R11: value 100k -> 27k
- R12: value 4.7k -> 27k
- R13: value 10k -> 27k
- R14: value 1k -> 10k
- R15: value 56k -> 20k
- R16: value 30k -> 220
- R17: value 10k -> 2k
- R18: value 100k -> 9.1k
- R19: value 6.8k -> 68k
- R20: value 2.2k -> 220
- R21: value 1k -> 2k
- R22: value 1k -> 9.1k
- R4: value 39 -> 1k
- R41: value 180 -> 82
- R42: value 180 -> 100
- R6, R7: device RFiD:R0402 -> RFiD:R0603
- R9: value 56k -> 3.9k
- U1: value ATXMEGA8E5-AU -> SAMD20E14A-AUT
- moved R21 162.5 mm to (70.0, 213.2), flipped to the top, turned to 90 degrees
- moved R20 160.5 mm to (60.4, 213.2), turned to 90 degrees
- moved C29 159.8 mm to (65.2, 213.2), flipped to the top, turned to 90 degrees
- moved R19 158.7 mm to (50.8, 213.2), turned to 90 degrees
- moved C28 156.8 mm to (55.6, 213.2), flipped to the top, turned to 90 degrees
- moved C24 156.0 mm to (31.6, 213.2), flipped to the top
- moved R18 155.8 mm to (26.8, 213.2), turned to 90 degrees
- moved C27 153.7 mm to (46.0, 213.2), flipped to the top, turned to 90 degrees
- moved R22 153.7 mm to (79.6, 207.6), turned to 90 degrees
- moved C25 150.4 mm to (36.4, 213.2), turned to 90 degrees
- moved R16 149.2 mm to (17.2, 213.2), turned to 90 degrees
- moved C26 148.8 mm to (41.2, 213.2), turned to 90 degrees
- moved R17 147.9 mm to (22.0, 213.2), turned to 90 degrees
- moved TOUCH-C 23.8 mm to (32.2, 39.8), turned to 90 degrees
- moved R23 21.4 mm to (25.2, 23.5), flipped to the top, turned to 0 degrees
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Connections:
- removed net LED-ACT: LED1.1, U1.23
- removed net N$1: D1.C, D2.C, L2.P$2
- removed net PDI_CLOCK: PROG/DBG.3, R23.1, U1.8
- removed net PDI_DATA: PROG/DBG.2, U1.7
- removed net PSK-CLK: U1.11, U1.24
- removed net USART-RXD0: D6.3, R38.1, U1.22
- removed net USART-TXD0: R32.2, U1.21
- new net D0/TX/CLK: R32.2, U1.20
- new net LED-GREEN-CTRL: LED2.1, U1.16
- new net LED-RED-CTRL: LED2.3, U1.17
- new net N$47: C2.1, U1.29
- new net N$59: Q2.2, R46.2
- new net N$60: Q3.E, R47.1
- new net N$63: C44.1, R21.2, R22.2, R48.2
- new net N$64: C45.1, IC2.2, R22.1
- new net N$65: C45.2, IC2.1, IC2.6, R48.1
- new net N$66: IC2.5, R49.2, R50.1
- new net N$69: C46.1, R51.1
- new net N$70: C47.2, C48.2, R51.2, R52.2
- new net N$71: C48.1, C49.1, IC2.8, R53.2
- new net N$72: C47.1, IC2.9, R53.1
- new net N$73: C49.2, R54.2
- new net N$74: C50.2, C51.2, R54.1, R55.2
- new net N$75: C51.1, IC2.13, R56.2
- new net OUT1: C26.2, C46.2, IC1.6, IC1.7, R14.2
- new net RESET: JP1.4, R23.1, U1.26
- new net SWDCLK: JP1.3
- new net SWDIO: JP1.2
- new net USART-RX: D6.3, R38.1, U1.19
- net +12V: now also C52.1, C53.1, D1.C, D2.C, IC1.4, Q2.3; no longer C18.1, L2.P$1, R4.2
- net +3V3: now also JP1.1, U1.3, U1.30; no longer PROG/DBG.1, U1.17, U1.6
- net +5V: now also IC1.12, IC2.10, IC2.12, IC2.3, R15.1, R50.2
- net ASK-FSK: now also IC2.7, R49.1, U1.14; no longer C21.1, R16.2, R17.2, U1.26
- net BUZZER: now also U1.1; no longer U1.25
- net CARD-PRES: now also U1.24; no longer U1.19
- net D1/DATA: now also U1.23; no longer U1.16
- net GND: now also C25.2, C29.2, C43.2, C44.2, C52.2, C53.2, IC1.11, JP1.5, R52.1, R55.1, U1.10, U1.28; no longer C19.2, C21.2, C22.2, C27.2, LED1.4, PROG/DBG.4, R17.1, R20.1, R21.2, R22.1, U1.1, U1.18
- net LED-INPUT: now also U1.18; no longer U1.9
- net MIFARE-IRQ: no longer U1.15
- net MIFARE-RST: now also U1.2; no longer U1.20
- net MIFARE-SCL: now also U1.22; no longer U1.27
- net MIFARE-SDA: now also U1.21; no longer U1.28
- net N$10: now also C18.1; no longer Q2.3
- net N$11: now also R46.1, R47.2; no longer Q2.2, Q3.E
- net N$15: now also C19.2, IC1.2, R4.2, R9.1; no longer C27.1, IC2.12, R12.2
- net N$16: now also IC1.3; no longer IC2.10, IC2.3
- net N$17: now also C19.1, C22.2, IC1.1, R10.1, R9.2; no longer C20.2, IC2.7, R15.2, R16.1
- net N$19: now also C21.1, R10.2, R11.1; no longer IC2.6, R14.1, R15.1
- net N$2: now also U4.15; no longer U4.12
- net N$20: now also C23.2, R12.1, R13.1; no longer R14.2
- net N$21: now also C20.2, C21.2, IC1.8, IC1.9, R12.2; no longer C23.2, IC2.1, R9.1
- net N$22: now also C26.1, R16.2; no longer C19.1, IC2.5, R13.1
- net N$23: now also C23.1, IC1.5, R11.2; no longer C28.2, C29.2, R21.1
- net N$24: now also R16.1, R17.2; no longer R10.2
- net N$25: now also C25.1, R17.1, R18.2, R19.2; no longer C23.1, IC2.2, R10.1, R9.2
- net N$26: now also IC1.10, R14.1, R15.2; no longer C25.2, C26.2, R22.2
- net N$27: now also C27.2, IC1.13, R18.1; no longer C25.1, IC2.9, R11.1
- net N$28: now also C27.1, IC1.14, R19.1; no longer IC2.13, R18.1
- net N$29: now also C28.2, R20.1; no longer C26.1, IC2.8, R11.2, R12.1
- net N$30: now also R20.2, R21.1; no longer IC2.14, R18.2, R19.1
- net N$4: now also U4.12; no longer U4.15
- net N$40: now also C43.1, U1.9; no longer C2.1, U1.32
- net N$52: now also LED2.4; no longer LED1.3
- net N$53: now also LED2.2; no longer LED1.2
- net PSK: now also C50.1, IC2.14, R56.1, U1.15; no longer R19.2, R20.2, U1.10
- net RELE: now also U1.32; no longer U1.12
- net TOUCH-C1: now also U1.8; no longer U1.31
- net TOUCH-C2: now also U1.11; no longer U1.30
- net TOUCH-C3: now also U1.12; no longer U1.29
- net TOUCH-L1: now also U1.4; no longer U1.5
- net TOUCH-L2: now also U1.5; no longer U1.4
- net TOUCH-L3: now also U1.6; no longer U1.3
- net TOUCH-L4: now also U1.7; no longer U1.2
Routing:
- net +3V3: track 157.4 -> 0.00 mm, vias 10 -> 0
- net +12V: track 113.8 -> 0.00 mm, vias 4 -> 0
- net +5V: track 76.0 -> 0.00 mm, vias 6 -> 0
- net ASK-FSK: track 49.3 -> 0.00 mm, vias 2 -> 0
- net PSK: track 34.6 -> 0.00 mm, vias 2 -> 0
- net RELE: track 31.6 -> 0.00 mm, vias 2 -> 0
- net LED-ACT: track 28.1 -> 0.00 mm, vias 2 -> 0
- net MIFARE-RST: track 27.7 -> 0.00 mm, vias 1 -> 0
- net MIFARE-IRQ: track 22.9 -> 0.00 mm, vias 1 -> 0
- net BUZZER: track 20.8 -> 0.00 mm, vias 2 -> 0
- net LED-INPUT: track 24.6 -> 3.94 mm, vias 1 -> 0
- net N$16: track 20.3 -> 0.00 mm
- net PDI_CLOCK: track 18.9 -> 0.00 mm, vias 1 -> 0
- net 125KHZ-ANTENA: track 14.3 -> 0.00 mm, vias 1 -> 0
- net N$46: track 16.8 -> 2.66 mm, vias 1 -> 0
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- removed copper zone on layer 1, net +12V
- removed copper zone on layer 1, net +3V3
- removed copper zone on layer 1, net +5V
- removed copper zone on layer 1, net GND

Commit message: Mudanças de packages e início de roteamento.
Parts:
- removed U2: AP1117IE33G-13, RFiD:SOT223-3L
- added U5: LP2985-33DBVR, RFiD:SOT-23-5
- C1, C4: device RFiD:C1206 -> RFiD:C0805
- C6, C7: value 10uF -> 4.7uF; device RFiD:C1206 -> RFiD:C0603
- moved C53 207.8 mm to (16.8, 62.9), flipped to the bottom, turned to 180 degrees
- moved C52 197.4 mm to (40.6, 51.3), turned to 0 degrees
- moved C45 168.9 mm to (26.6, 50.7), flipped to the bottom, turned to 180 degrees
- moved C44 166.5 mm to (26.5, 53.9)
- moved R48 166.4 mm to (27.3, 51.3)
- moved R21 166.3 mm to (24.2, 53.3), turned to 0 degrees
- moved R22 165.3 mm to (25.7, 51.3)
- moved C28 164.8 mm to (19.0, 52.5), flipped to the bottom, turned to 180 degrees
- moved R20 164.6 mm to (21.4, 53.3), flipped to the bottom, turned to 180 degrees
- moved C29 163.6 mm to (24.2, 54.8), turned to 0 degrees
- moved R19 162.0 mm to (19.8, 54.2), turned to 0 degrees
- moved C27 160.9 mm to (19.0, 54.6), flipped to the bottom, turned to 0 degrees
- moved R18 157.1 mm to (19.0, 56.3), flipped to the bottom, turned to 180 degrees
- moved C25 157.0 mm to (21.1, 56.9), flipped to the bottom
- moved C24 156.7 mm to (22.5, 56.8), turned to 0 degrees
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Connections:
- net +12V: no longer C6.1, U2.3
- net +3V3: now also U5.5; no longer U2.2, U2.4
- net +5V: now also C6.1, U5.1, U5.3
- net ASK-FSK: now also U1.15; no longer U1.14
- net GND: now also U5.2; no longer U2.1
- net PSK: now also U1.14; no longer U1.15
- net RELE: now also U1.25; no longer U1.32
Routing:
- net GND: track 0.00 -> 53.1 mm, vias 0 -> 37
- net +5V: track 0.00 -> 51.4 mm, vias 0 -> 4
- net OUT1: track 0.00 -> 21.9 mm
- net ASK-FSK: track 0.00 -> 19.9 mm, vias 0 -> 1
- net 125KHZ-ANTENA: track 0.00 -> 18.9 mm
- net PSK: track 0.00 -> 18.0 mm, vias 0 -> 1
- net LED-RED-CTRL: track 0.00 -> 17.8 mm, vias 0 -> 2
- net +12V: track 0.00 -> 17.3 mm
- net TOUCH-C3: track 0.00 -> 16.2 mm
- net LED-INPUT: track 3.94 -> 19.0 mm
- net LED-GREEN-CTRL: track 0.00 -> 15.0 mm
- net MIFARE-SDA: track 0.00 -> 13.5 mm, vias 0 -> 2
- net USART-RX: track 2.09 -> 15.5 mm
- net TOUCH-C2: track 0.00 -> 13.4 mm
- net +3V3: track 0.00 -> 12.7 mm
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Other:
- board size 34.5 x 67 mm -> 34.5 x 68 mm

Commit message: Mais progressos, próximo do final.
Parts:
- added D: LL4148, RFiD:SOD80C
- C42: device RFiD:C0805 -> RFiD:C0402
- C43: device RFiD:C0402 -> RFiD:C0603
- moved C52 17.1 mm to (23.5, 50.3), turned to 180 degrees
- moved C42 11.0 mm to (21.7, 28.9), turned to 180 degrees
- moved L6 10.2 mm to (20.5, 30.6)
- moved C3 7.14 mm to (23.2, 21.9), turned to 180 degrees
- moved C2 4.92 mm to (22.5, 25.2)
- moved R23 4.71 mm to (29.7, 22.1), flipped to the bottom, turned to 90 degrees
- moved Q8 3.30 mm to (4.80, 8.40)
- moved R27 2.86 mm to (21.9, 12.2), flipped to the bottom
- moved R45 2.61 mm to (8.20, 9.50), turned to 0 degrees
- moved C46 1.32 mm to (20.0, 48.7)
- moved C9 1.30 mm to (23.5, 20.5), turned to 180 degrees
- moved R50 1.20 mm to (22.1, 46.9)
- moved C41 1.10 mm to (22.5, 13.7), turned to 0 degrees
- moved R48 1.00 mm to (28.3, 51.3)
- moved R22 0.90 mm to (26.6, 51.3)
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Connections:
- net +12V: now also D.C
- net MIFARE-RST: now also U1.27; no longer U1.2
- net N$48: now also D.A
- net SWDCLK: now also U1.31
- net SWDIO: now also U1.32
Routing:
- net +12V: track 17.3 -> 103.7 mm, vias 0 -> 4
- net +5V: track 51.4 -> 82.5 mm, vias 4 -> 6
- net RESET: track 0.00 -> 27.3 mm
- net RELE: track 0.00 -> 20.7 mm
- net BUZZER: track 0.00 -> 18.6 mm, vias 0 -> 2
- net MIFARE-RST: track 0.00 -> 18.4 mm, vias 0 -> 2
- net SWDCLK: track 0.00 -> 14.0 mm
- net SWDIO: track 0.00 -> 10.1 mm
- net +3V3: track 12.7 -> 22.7 mm, vias 0 -> 1
- net GND: track 53.1 -> 62.0 mm, vias 37 -> 47
- net N$40: track 0.00 -> 6.85 mm, vias 0 -> 1
- net N$37: track 0.00 -> 5.47 mm, vias 0 -> 1
- net MIFARE-RX: track 0.00 -> 4.11 mm, vias 0 -> 1
- net N$31: track 2.23 -> 5.15 mm, vias 0 -> 1
- net N$47: track 0.00 -> 2.13 mm, vias 0 -> 1
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
Commit message: Roteamento finalizado. Verificar posiconamento.
Espessuras de trilhas precisam ser revisadas.
Parts:
- moved R52 0.78 mm to (21.2, 42.1), turned to 0 degrees
- moved C9 0.71 mm to (22.8, 20.6)
- moved D2 0.70 mm to (5.60, 43.6)
- moved QZ1 0.70 mm to (24.2, 18.0)
- moved R32 0.70 mm to (11.4, 29.1)
- moved R38 0.61 mm to (4.70, 34.9)
- moved R28 0.61 mm to (4.70, 36.3)
- moved L4 0.58 mm to (16.3, 7.80)
- moved L5 0.58 mm to (20.0, 7.80)
- moved R40 0.50 mm to (5.40, 38.2)
- moved R39 0.41 mm to (4.70, 33.4)
- moved C6 0.30 mm to (7.90, 45.2)
- moved R36 0.22 mm to (4.70, 27.4)
- moved C5 0.22 mm to (24.8, 15.3)
- moved U5 0.20 mm to (11.0, 45.1)
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Routing:
- net +3V3: track 22.7 -> 124.6 mm, vias 1 -> 12
- net +5V: track 82.5 -> 108.6 mm, vias 6 -> 11
- net +12V: track 103.7 -> 127.3 mm, vias 4 -> 10
- net LED-INPUT: track 19.0 -> 20.7 mm
- net MIFARE-TX2: track 5.88 -> 6.68 mm
- net N$28: track 5.89 -> 6.49 mm
- net N$3: track 8.80 -> 8.22 mm
- net N$31: track 5.15 -> 4.64 mm
- net MIFARE-TX1: track 6.60 -> 7.10 mm
- net GND: track 62.0 -> 62.1 mm, vias 47 -> 48
- net N$59: vias 0 -> 1

Commit message: Versão da leitora com as alterações solicitadas e outras.
Parts:
- added ASK/FSK, PSK, TP1, TP2, TP3, TP4, TP5, TP6, TP9: TESTPOINT, RFiD:TESTPOINT
- added C54: 100nF, RFiD:C0402
- added C55: 10nF, RFiD:C0402
- added R57, R58: 470, RFiD:R0402
- D3, D4: value BAV199 -> BAV99
- moved C46 5.72 mm to (21.9, 54.1)
- moved R41 2.20 mm to (16.5, 46.5), flipped to the bottom, turned to 90 degrees
- moved R42 2.20 mm to (18.0, 46.5), flipped to the bottom, turned to 270 degrees
- moved C17 0.90 mm to (13.7, 65.1)
- moved D4 0.90 mm to (16.3, 66.1)
- moved R8 0.90 mm to (16.5, 66.1)
- moved R50 0.85 mm to (22.7, 47.5), turned to 270 degrees
- moved C9 0.42 mm to (22.5, 20.9)
- moved C5 0.30 mm to (24.8, 15.0)
- moved R22 0.30 mm to (26.3, 51.3)
- moved R14 0.30 mm to (13.5, 59.5)
- moved R15 0.20 mm to (12.9, 57.6)
- moved R5 0.20 mm to (29.7, 45.1)
- renumbered D to D7, JP1 to SWD
Connections:
- new net V+: C54.1, C55.1, IC1.12, IC2.10, IC2.12, IC2.3, R15.1, R50.2, R57.2, R58.2
- net +12V: now also R57.1
- net +5V: no longer IC1.12, IC2.10, IC2.12, IC2.3, R15.1, R50.2
- net ASK-FSK: now also ASK/FSK.P$1
- net GND: now also C54.2, C55.2, R58.1
- net N$16: now also TP1.P$1
- net N$17: now also TP2.P$1
- net N$26: now also TP4.P$1
- net N$28: now also TP5.P$1
- net N$65: now also TP6.P$1
- net N$71: now also PSK.P$1
- net OUT1: now also TP3.P$1
- net PSK: now also TP9.P$1
Routing:
- net +5V: track 108.6 -> 71.3 mm, vias 11 -> 8
- net V+: track 0.00 -> 37.0 mm, vias 0 -> 3
- net N$69: track 1.70 -> 8.59 mm
- net +12V: track 127.3 -> 133.8 mm
- net +3V3: track 124.6 -> 121.6 mm, vias 12 -> 13
- net N$71: track 6.73 -> 9.56 mm
- net N$66: track 6.53 -> 4.37 mm
- net PSK: track 17.0 -> 19.0 mm
- net 125KHZ-ANTENA: track 16.9 -> 18.7 mm
- net N$65: track 11.7 -> 13.3 mm
- net ASK-FSK: track 19.8 -> 21.3 mm
- net N$28: track 6.49 -> 7.92 mm
- net N$17: track 8.26 -> 9.66 mm
- net OUT1: track 21.8 -> 20.4 mm
- net TOUCH-C3: track 15.2 -> 16.5 mm
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Other:
- board text added: "!RESET"
- board text added: "+3V3"
- board text added: "GND"
- board text added: "SWD"
- board text added: "SWDCLK"
- board text added: "SWDIO"
- board text added: "U3"

Commit message: Próximo RC de versão de versão final.
Parts:
- added SJ?1: SOLDERBRIDGE, RFiD:SOLDERBRIDGE
Connections:
- new net N$77: R44.2, SG1.+, SJ?1.2
- net +12V: now also SJ?1.1
- net +3V3: now also SJ?1.3; no longer R44.2, SG1.+
Routing:
- net +12V: track 133.8 -> 160.3 mm
- net N$77: track 0.00 -> 7.59 mm
- net +3V3: track 121.6 -> 117.2 mm
Other:
- board text added: "+12V"
- board text added: "AGN"
- board text added: "AN"
- board text added: "BUZZ"
- board text added: "DN"
- board text added: "www.controlid.com.br"

Commit message: Nova versão do leitor. Aguardando revisão.
Parts:
- removed C43: 4.7uF, RFiD:C0603
- removed COM: COM, RFiD:HOLE
- removed D7: LL4148, RFiD:SOD80C
- removed L6: BEAD, RFiD:R0402
- removed NC: NC, RFiD:HOLE
- removed NO: NO, RFiD:HOLE
- removed Q8: BC847ALT1SMD, RFiD:SOT23
- removed R45: 2.2k, RFiD:R0402
- removed RL1: RELE, RFiD:RELE
- removed TOUCH-C, TOUCH-L: (no value), pinhead:1X04
- removed TP9: TESTPOINT, RFiD:TESTPOINT
- added TP8: TESTPOINT, RFiD:TESTPOINT
- moved D6 23.9 mm to (8.30, 11.1)
- moved D5 23.6 mm to (8.30, 15.0)
- moved R39 22.3 mm to (4.80, 11.1)
- moved R38 22.1 mm to (4.80, 12.8)
- moved R40 21.5 mm to (4.80, 16.7), turned to 180 degrees
- moved R28 21.3 mm to (4.80, 15.0)
- moved LED-IN 20.0 mm to (2.10, 16.2)
- moved MODE-SEL 20.0 mm to (2.10, 13.7)
- moved C38 17.0 mm to (6.70, 8.20), turned to 0 degrees
- moved C9 16.1 mm to (23.7, 4.80), flipped to the bottom, turned to 270 degrees
- moved X2 14.9 mm to (3.40, 5.70), turned to 270 degrees
- moved R25 14.8 mm to (6.70, 6.70), turned to 180 degrees
- moved QZ1 13.9 mm to (26.0, 4.20)
- moved C40 13.8 mm to (9.30, 3.10), turned to 180 degrees
- moved PSK 13.4 mm to (27.6, 27.3)
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Connections:
- removed net N$40: C42.1, C43.1, L6.1, U1.9
- removed net N$48: D7.A, Q8.3, RL1.1
- removed net N$49: Q8.1, R45.1
- removed net N$56: NO.P$1, RL1.3
- removed net N$57: NC.P$1, RL1.4
- removed net N$58: COM.P$1, RL1.2
- removed net RELE: R45.2, U1.25
- removed net TOUCH-C1: TOUCH-C.1, U1.8
- removed net TOUCH-C2: TOUCH-C.2, U1.11
- removed net TOUCH-C3: TOUCH-C.3, U1.12
- removed net TOUCH-L1: TOUCH-L.1, U1.4
- removed net TOUCH-L2: TOUCH-L.2, U1.5
- removed net TOUCH-L3: TOUCH-L.3, U1.6
- removed net TOUCH-L4: TOUCH-L.4, U1.7
- net +12V: no longer D7.C, RL1.5
- net +3V3: now also C42.1, U1.9; no longer L6.2, U1.3
- net 125KHZ-ANTENA: now also U1.1; no longer U1.13
- net ASK-FSK: now also U1.3; no longer U1.15
- net BUZZER: now also U1.24; no longer U1.1
- net CARD-PRES: now also U1.13; no longer U1.24
- net D0/TX/CLK: now also U1.11; no longer U1.20
- net D1/DATA: now also U1.12; no longer U1.23
- net GND: no longer C43.2, Q8.2, TOUCH-C.4
- net LED-GREEN-CTRL: now also U1.5; no longer U1.16
- net LED-INPUT: now also U1.14; no longer U1.18
- net LED-RED-CTRL: now also U1.4; no longer U1.17
- net MIFARE-RST: now also U1.17; no longer U1.27
- net MIFARE-SCL: now also U1.21; no longer U1.22
- net MIFARE-SDA: now also U1.22; no longer U1.21
- net N$2: now also U4.12; no longer U4.15
- net N$38: now also X2.2; no longer X2.1
- net N$39: now also X2.1; no longer X2.2
- net N$4: now also U4.15; no longer U4.12
- net N$71: now also TP8.P$1; no longer PSK.P$1
- net PSK: now also PSK.P$1, U1.2; no longer TP9.P$1, U1.14
- net USART-RX: now also U1.15; no longer U1.19
Routing:
- net RELE: track 20.7 -> 0.00 mm
- net +3V3: track 117.2 -> 134.3 mm, vias 13 -> 15
- net TOUCH-C3: track 16.5 -> 0.00 mm
- net BUZZER: track 18.6 -> 2.11 mm, vias 2 -> 0
- net +12V: track 160.3 -> 146.3 mm, vias 10 -> 11
- net TOUCH-C2: track 13.4 -> 0.00 mm
- net MIFARE-RST: track 18.2 -> 4.89 mm
- net N$56: track 11.6 -> 0.00 mm
- net TOUCH-C1: track 9.45 -> 0.00 mm
- net GND: track 63.2 -> 54.1 mm, vias 52 -> 51
- net N$57: track 8.98 -> 0.00 mm
- net RESET: track 27.5 -> 18.7 mm
- net TOUCH-L4: track 8.52 -> 0.00 mm
- net TOUCH-L1: track 7.94 -> 0.00 mm
- net TOUCH-L3: track 7.80 -> 0.00 mm
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Other:
- board size 34.5 x 68 mm -> 34.5 x 56.7 mm
- board text added: "ASK"
- board text added: "FSK"
