File: Hardware/PAINEL.brd (EAGLE design)
At the start: 113.5 x 123.4 mm, 1002 parts, among them IC1 TL084, IC10 TL084, IC11 TL084, IC12 TL084, IC2 TL084, IC3 TL084, IC4 TL084, IC5 TL084, IC6 TL084, IC7 TL084, IC8 TL084, IC9 TL084, Q1 DMN3404, Q10 MMBT4401, Q11 MMBT4401, Q12 DMN3404, Q13 MMBT4403, Q14 MMBT4401, Q15 MMBT4401, Q16 MMBT4401, Q17 MMBT4401, Q18 MMBT4401, Q19 DMN3404, Q2 MMBT4401, Q20 MMBT4403, Q21 MMBT4401, Q22 MMBT4401, Q23 MMBT4401, Q24 MMBT4401, Q25 MMBT4401, Q26 DMN3404, Q27 MMBT4403, Q28 MMBT4401, Q29 MMBT4401, Q3 MMBT4403, Q30 MMBT4401, Q31 MMBT4401, Q32 MMBT4401, Q33 DMN3404, Q34 MMBT4403, Q35 MMBT4401, Q36 MMBT4401, Q37 MMBT4401, Q38 MMBT4401, Q39 MMBT4401, Q4 MMBT4401, Q40 DMN3404, Q41 MMBT4403, Q42 MMBT4401, Q5 MMBT4401, Q6 MMBT4401, Q7 MMBT4401, Q8 MMBT4401, Q9 MMBT4401, U1 LP2985-33DBVR, U10 MFRC52202HN1, U11 SAMD20E14A-AUT, U12 LP2985-33DBVR, U13 TLV1117-50CDCYR, U14 MFRC52202HN1, U15 SAMD20E14A-AUT, U16 LP2985-33DBVR, U17 TLV1117-50CDCYR, U18 MFRC52202HN1, U19 SAMD20E14A-AUT, U2 TLV1117-50CDCYR, U20 LP2985-33DBVR, U21 TLV1117-50CDCYR, U22 MFRC52202HN1, U23 SAMD20E14A-AUT, U24 LP2985-33DBVR, U3 SAMD20E14A-AUT, U4 MFRC52202HN1, U5 TLV1117-50CDCYR, U6 MFRC52202HN1, U7 SAMD20E14A-AUT, U8 LP2985-33DBVR, U9 TLV1117-50CDCYR, X1 ANTENA, X10 MIFARE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

Commit message: Arquivos panelizados. Fim. Conforme enviado para Joy.
Parts:
- C101, C104, C118, C165, C168, C182, C229, C232, C246, C29, C293, C296, C310, C35, C357, C360, C374, C45: value 0.1u -> F:0.1uP:10n
- C102, C106, C119, C166, C170, C183, C230, C234, C247, C294, C298, C311, C32, C358, C362, C375, C39, C44: value F:P:100p -> F:1nP:100p
- C103, C105, C120, C167, C169, C184, C231, C233, C248, C295, C297, C31, C312, C359, C361, C376, C38, C43: value F:P:68p -> F:220pP:68p
- C113, C177, C21, C241, C305, C369: device RFiD:C0805 -> RFiD:C0603
- C114, C178, C22, C242, C306, C370: device RFiD:C1812 -> RFiD:C1812S
- C115, C133, C179, C197, C243, C261, C27, C28, C307, C325, C371, C69: device RFiD:C1206 -> RFiD:C1206S
- R105, R108, R125, R169, R172, R189, R21, R233, R236, R253, R297, R300, R317, R35, R361, R364, R381, R40: value F:P:5.6k -> F:5.1kP:5.6k
- R106, R109, R127, R170, R173, R191, R23, R234, R237, R255, R298, R301, R319, R36, R362, R365, R383, R39: value F:P:5.1k -> F:7.5kP:5.1k
- R107, R110, R126, R171, R174, R190, R235, R238, R254, R27, R299, R302, R31, R318, R363, R366, R382, R41: value F:P:270k -> F:180kP:270k
- R131, R15, R195, R259, R323, R67: device RFiD:R1206 -> RFiD:R1206S
- R152, R216, R280, R344, R53, R88: value 150 -> 130
- R153, R217, R281, R345, R54, R89: value 150 -> 120
- U1, U12, U16, U20, U24, U8: value LP2985-33DBVR -> TLV71333PDBVR
- U13, U17, U2, U21, U5, U9: value TLV1117-50CDCYR -> NCP1117LPST50T3G
- X10, X12, X2, X4, X6, X8: device RFiD:22-23-2021 -> RFiD:ANTENNA
- moved C133 13.7 mm to (53.5, 54.0), turned to 210 degrees
- moved C197 13.7 mm to (53.5, 110.7), turned to 210 degrees
- moved C261 13.7 mm to (88.0, 54.0), turned to 210 degrees
- moved C28 13.7 mm to (19.0, 54.0), turned to 210 degrees
- moved C325 13.7 mm to (88.0, 110.7), turned to 210 degrees
- moved C69 13.7 mm to (19.0, 110.7), turned to 210 degrees
- moved FID10 11.3 mm to (91.5, 16.6)
- moved FID3 11.3 mm to (22.5, 16.6)
- moved FID6 11.3 mm to (57.0, 16.6)
- moved FID12 11.3 mm to (91.5, 73.3)
- moved FID4 11.3 mm to (22.5, 73.3)
- moved FID8 11.3 mm to (57.0, 73.3)
- moved C307 9.13 mm to (90.8, 49.8), turned to 210 degrees
- moved C371 9.13 mm to (90.8, 106.5), turned to 210 degrees
- moved C179 9.13 mm to (56.4, 49.8), turned to 210 degrees
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Routing:
- net N$183: track 3.92 -> 16.5 mm, vias 0 -> 2
- net N$14: track 3.92 -> 16.5 mm, vias 0 -> 2
- net N$317: track 3.92 -> 16.5 mm, vias 0 -> 2
- net N$250: track 3.92 -> 16.5 mm, vias 0 -> 2
- net N$116: track 3.92 -> 16.5 mm, vias 0 -> 2
- net N$384: track 3.92 -> 16.5 mm, vias 0 -> 2
- net +12V4: track 118.0 -> 107.1 mm, vias 7 -> 14
- net +12V3: track 118.0 -> 107.1 mm, vias 7 -> 14
- net +12V2: track 118.0 -> 107.1 mm, vias 7 -> 14
- net +12V1: track 118.0 -> 107.1 mm, vias 7 -> 14
- net +12V5: track 118.0 -> 107.1 mm, vias 7 -> 14
- net +12V: track 118.0 -> 107.1 mm, vias 7 -> 14
- net N$5: track 12.9 -> 8.41 mm
- net N$277: track 12.9 -> 8.41 mm
- net N$73: track 12.9 -> 8.41 mm
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- added copper zone on layer 16, net +12V
- added copper zone on layer 16, net +12V1
- added copper zone on layer 16, net +12V2
- added copper zone on layer 16, net +12V3
- added copper zone on layer 16, net +12V4
- added copper zone on layer 16, net +12V5
Other:
- outline, holes or cut-outs redrawn
- board text added: "CONTROL ID - LEITORRF V4"
- board text added: "D1"
- board text added: "D3"
- board text added: "IC1"
- board text added: "IC2"
- board text added: "LEITOR"
- board text added: "RF"
- board text added: "Rev. 4"
- board text added: "U4"
- board text removed: "CONTROL ID - LEITORRF V3"
