File: Hardware/PAINELVIRGEM.brd (EAGLE design)
At the start: 113.5 x 123.4 mm, 6 parts

Commit message: Arquivos panelizados. Fim. Conforme enviado para Joy.
Other:
- board text added: "CONTROL ID - LEITORRF V4"
- board text removed: "CONTROL ID - LEITORRF V3"
Changed lines of the file:
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@@
 <grid distance="0.1" unitdist="mm" unit="mm" style="lines" multiple="1" display="yes" altdistance="56.7" altunitdist="mm" altunit="mm"/>
 <layers>
-<layer number="1" name="Top" color="4" fill="1" visible="no" active="yes"/>
+<layer number="1" name="Top" color="4" fill="1" visible="yes" active="yes"/>
 <layer number="2" name="Route2" color="1" fill="3" visible="no" active="no"/>
 <layer number="3" name="Route3" color="4" fill="3" visible="no" active="no"/>
-<layer number="4" name="Route4" color="1" fill="4" visible="no" active="yes"/>
-<layer number="5" name="Route5" color="4" fill="4" visible="no" active="yes"/>
+<layer number="4" name="Route4" color="1" fill="4" visible="yes" active="yes"/>
+<layer number="5" name="Route5" color="4" fill="4" visible="yes" active="yes"/>
 <layer number="6" name="Route6" color="1" fill="8" visible="no" active="no"/>
 <layer number="7" name="Route7" color="4" fill="8" visible="no" active="no"/>
@@
 <layer number="14" name="Route14" color="1" fill="6" visible="no" active="no"/>
 <layer number="15" name="Route15" color="4" fill="6" visible="no" active="no"/>
-<layer number="16" name="Bottom" color="1" fill="1" visible="no" active="yes"/>
-<layer number="17" name="Pads" color="2" fill="1" visible="no" active="yes"/>
-<layer number="18" name="Vias" color="2" fill="1" visible="no" active="yes"/>
-<layer number="19" name="Unrouted" color="6" fill="1" visible="no" active="yes"/>
+<layer number="16" name="Bottom" color="1" fill="1" visible="yes" active="yes"/>
+<layer number="17" name="Pads" color="2" fill="1" visible="yes" active="yes"/>
+<layer number="18" name="Vias" color="2" fill="1" visible="yes" active="yes"/>
+<layer number="19" name="Unrouted" color="6" fill="1" visible="yes" active="yes"/>
 <layer number="20" name="Dimension" color="15" fill="1" visible="yes" active="yes"/>
-<layer number="21" name="tPlace" color="7" fill="1" visible="no" active="yes"/>
+<layer number="21" name="tPlace" color="7" fill="1" visible="yes" active="yes"/>
 <layer number="22" name="bPlace" color="7" fill="1" visible="yes" active="yes"/>
 <layer number="23" name="tOrigins" color="15" fill="1" visible="yes" active="yes"/>
@@
 <wire x1="103.5" y1="0" x2="103.5" y2="113.4" width="0" layer="20"/>
 <wire x1="0" y1="113.4" x2="103.5" y2="113.4" width="0" layer="20"/>
-<text x="-1.3" y="34.5" size="2.1844" layer="21" font="vector" ratio="14" rot="R90">CONTROL ID - LEITORRF V3</text>
-<text x="107.1" y="34.5" size="2.1844" layer="21" font="vector" ratio="14" rot="R90">CONTROL ID - LEITORRF V3</text>
-<text x="-1.3" y="78.9" size="2.1844" layer="22" font="vector" ratio="14" rot="SMR270">CONTROL ID - LEITORRF V3</text>
-<text x="107.1" y="79" size="2.1844" layer="22" font="vector" ratio="14" rot="SMR270">CONTROL ID - LEITORRF V3</text>
+<text x="-1.3" y="34.5" size="2.1844" layer="21" font="vector" ratio="14" rot="R90">CONTROL ID - LEITORRF V4</text>
+<text x="107.1" y="34.5" size="2.1844" layer="21" font="vector" ratio="14" rot="R90">CONTROL ID - LEITORRF V4</text>
+<text x="-1.3" y="78.9" size="2.1844" layer="22" font="vector" ratio="14" rot="SMR270">CONTROL ID - LEITORRF V4</text>
+<text x="107.1" y="79" size="2.1844" layer="22" font="vector" ratio="14" rot="SMR270">CONTROL ID - LEITORRF V4</text>
 </plain>
 <attributes>
